File: Ritsumori cup2026/Substrate/sentral board_1.0/sentral board_1.0.kicad_pcb (KiCad board)
At the start: 2 copper layers, 40.6 x 35.9 mm, 9 parts, among them J1 Conn_02x10_Odd_Even, J2 Conn_02x05_Counter_Clockwise, J3 Conn_01x04_Socket, J4 Conn_01x05_Socket, J5 Conn_01x02_Socket, J6 Conn_01x02_Socket, J7 Conn_01x02_Socket, J8 Conn_01x02_Socket, J9 Conn_01x04_Socket

Commit message: Auto Backup: 2026/02/19 18:25:14.96
Parts:
- moved J6 36.0 mm to (183.0, 94.5), turned to 90 degrees
- moved J8 36.0 mm to (216.0, 109.0), turned to -90 degrees
- moved J5 35.2 mm to (183.0, 103.0), turned to 90 degrees
- moved J7 35.2 mm to (216.0, 90.8), turned to -90 degrees
Connections:
- J1 pad 1: UART2_TX_Angel -> GND
- J1 pad 10: Motor3_A -> Motor3_B
- J1 pad 11: UART4_RX_Camera -> UART4_TX_Camera
- J1 pad 12: Motor3_B -> Motor3_A
- J1 pad 13: +12V -> UART3_RX_IR
- J1 pad 14: Motor4_A -> Motor2_B
- J1 pad 15: +12V -> UART3_TX_IR
- J1 pad 16: Motor4_B -> Motor2_A
- J1 pad 17: VDD -> UART2_RX_Angel
- J1 pad 18: SW -> Motor1_B
- J1 pad 19: GND -> UART2_TX_Angel
- J1 pad 2: Motor1_A -> GND
- J1 pad 20: GND -> Motor1_A
- J1 pad 3: UART2_RX_Angel -> VDD
- J1 pad 4: Motor1_B -> SW
- J1 pad 5: UART3_TX_IR -> +12V
- J1 pad 6: Motor2_A -> Motor4_B
- J1 pad 7: UART3_RX_IR -> +12V
- J1 pad 8: Motor2_B -> Motor4_A
- J1 pad 9: UART4_TX_Camera -> UART4_RX_Camera
- J5 pad 1: Motor1_A -> Motor1_B
- J5 pad 2: Motor1_B -> Motor1_A
- J6 pad 1: Motor2_A -> Motor2_B
- J6 pad 2: Motor2_B -> Motor2_A
- J7 pad 1: Motor3_A -> Motor3_B
- J7 pad 2: Motor3_B -> Motor3_A
- J8 pad 1: Motor4_A -> Motor4_B
- J8 pad 2: Motor4_B -> Motor4_A
Routing:
- net Motor3_A: track 57.4 -> 10.7 mm
- net Motor3_B: track 55.1 -> 11.3 mm
- net Motor4_B: track 55.1 -> 19.7 mm, vias 1 -> 0
- net Motor4_A: track 55.0 -> 19.7 mm
- net Motor2_A: track 19.5 -> 54.6 mm, vias 0 -> 1
- net Motor1_B: track 7.62 -> 42.6 mm, vias 0 -> 1
- net Motor2_B: track 20.1 -> 54.2 mm
- net Motor1_A: track 7.63 -> 39.0 mm, vias 0 -> 1
- net UART3_TX_IR: track 8.37 -> 21.5 mm, vias 0 -> 2
- net VDD: track 66.9 -> 75.3 mm
- net UART3_RX_IR: track 8.38 -> 16.2 mm, vias 0 -> 2
- net UART4_TX_Camera: track 22.7 -> 15.2 mm
- net SW: track 36.1 -> 29.6 mm, vias 3 -> 0
- net UART2_TX_Angel: track 22.4 -> 27.6 mm, vias 0 -> 1
- net UART4_RX_Camera: track 12.6 -> 16.0 mm
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