File: Ritsumori cup2026/Substrate/sentral board_1.0/sentral board_1.0.kicad_pcb (KiCad board)
At the start: 2 copper layers, 40.6 x 35.9 mm, 9 parts, among them J1 Conn_02x10_Odd_Even, J2 Conn_02x05_Counter_Clockwise, J3 Conn_01x04_Socket, J4 Conn_01x05_Socket, J5 Conn_01x02_Socket, J6 Conn_01x02_Socket, J7 Conn_01x02_Socket, J8 Conn_01x02_Socket, J9 Conn_01x04_Socket

Commit message: Auto Backup: 2026/03/09 13:07:55.49
Connections:
- J3 pad 1: UART2_TX_Angel -> UART2_RX_Angel
- J3 pad 2: UART2_RX_Angel -> UART2_TX_Angel
- J4 pad 1: UART3_TX_IR -> UART3_RX_IR
- J4 pad 2: UART3_RX_IR -> UART3_TX_IR
Routing:
- net UART3_TX_IR: track 21.5 -> 19.2 mm
- net UART2_TX_Angel: track 27.6 -> 25.3 mm
- net UART3_RX_IR: track 16.2 -> 17.9 mm
- net GND: vias 33 -> 49
