File: Ritsumori cup2026/Substrate/IR board_1.0/IR board_1.0.kicad_pcb (KiCad board)
At the start: 2 copper layers, 100 x 100 mm, 33 parts, among them IC1 STM32F446RET6, J1 PC, J2 main, SW2 SW_Push, U1 TSSP4038, U10 TSSP4038, U11 TSSP4038, U12 TSSP4038, U13 TSSP4038, U14 TSSP4038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

Commit message: Auto Backup: 2026/03/09 13:07:55.49
Parts:
- renumbered NRST to SW1
Connections:
- IC1 pad 42: unconnected-(IC1-PA9-Pad42) -> USART1_TX_IR
- IC1 pad 43: USART1_TX_IR -> USART1_RX_IR
- IC1 pad 44: USART1_RX_IR -> unconnected-(IC1-PA11-Pad44)
Changed lines of the file:
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@@
 	(net 47 "unconnected-(IC1-PH0-OSC_IN-Pad5)")
 	(net 48 "unconnected-(IC1-PB14-Pad35)")
-	(net 49 "unconnected-(IC1-PA9-Pad42)")
+	(net 49 "unconnected-(IC1-PA11-Pad44)")
 	(net 50 "unconnected-(IC1-PA4-Pad20)")
 	(net 51 "unconnected-(IC1-PB9-Pad62)")
@@
 		(descr "J Lead 4.20mm x 3.20mm")
 		(tags "Switch")
-		(property "Reference" "NRST"
+		(property "Reference" "SW1"
 			(at 0 3.25 0)
 			(layer "F.SilkS")
@@
 			(layers "B.Cu" "B.Mask" "B.Paste")
 			(roundrect_rratio 0.25)
-			(net 49 "unconnected-(IC1-PA9-Pad42)")
+			(net 9 "USART1_TX_IR")
 			(pinfunction "PA9")
-			(pintype "passive+no_connect")
+			(pintype "passive")
 		)
 		(pad "43" smd roundrect
@@
 			(layers "B.Cu" "B.Mask" "B.Paste")
 			(roundrect_rratio 0.25)
-			(net 9 "USART1_TX_IR")
+			(net 8 "USART1_RX_IR")
 			(pinfunction "PA10")
 			(pintype "passive")
@@
 			(layers "B.Cu" "B.Mask" "B.Paste")
 			(roundrect_rratio 0.25)
-			(net 8 "USART1_RX_IR")
+			(net 49 "unconnected-(IC1-PA11-Pad44)")
 			(pinfunction "PA11")
-			(pintype "passive")
+			(pintype "passive+no_connect")
 		)
 		(pad "45" smd roundrect
@@
 			)
 		)
+		(property "LCSC" ""
+			(at 0 0 0)
+			(layer "B.SilkS")
+			(hide yes)
+			(effects
+				(font
+					(size 1.27 1.27)
+					(thickness 0.15)
+				)
+			)
+		)
 		(property ki_fp_filters "C_*")
 		(sheetname "ルート")
@@
 	)
 	(segment
-		(start 182.3 76.85)
-		(end 182.3 76.38)
+		(start 180.27 74.35)
+		(end 178.225 74.35)
 		(width 0.2)
 		(layer "B.Cu")
@@
 	(segment
 		(start 182.3 76.38)
-		(end 179.77 73.85)
+		(end 180.27 74.35)
 		(width 0.2)
 		(layer "B.Cu")
@@
 	)
 	(segment
-		(start 179.77 73.85)
-		(end 178.225 73.85)
+		(start 182.3 76.85)
+		(end 182.3 76.38)
 		(width 0.2)
 		(layer "B.Cu")
@@
 	)
 	(segment
-		(start 178.225 74.35)
-		(end 179.52 74.35)
+		(start 180.02 74.85)
+		(end 180.75 75.58)
 		(width 0.2)
 		(layer "B.Cu")
@@
 	)
 	(segment
-		(start 179.52 74.35)
-		(end 180.75 75.58)
+		(start 178.225 74.85)
+		(end 180.02 74.85)
 		(width 0.2)
 		(layer "B.Cu")
