File: Ritsumori cup2026/Substrate/power board_1.0/power board_1.0.kicad_pcb (KiCad board)
At the start: 2 copper layers, 66.7 x 63.9 mm, 23 parts, among them J1 Conn_01x02_Socket, J2 電圧計, J4 Conn_02x05_Counter_Clockwise, SW1 SW_Push_DPDT

Commit message: Auto Backup: 2026/03/09 13:07:55.49
Parts:
- renumbered D3 to 12V, D5 to 3.3V, D4 to 5V
Changed lines of the file:
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@@
 		(descr "LED SMD 0603 (1608 Metric), square (rectangular) end terminal, IPC_7351 nominal, (Body size source: http://www.tortai-tech.com/upload/download/2011102023233369053.pdf), generated with kicad-footprint-generator")
 		(tags "LED")
-		(property "Reference" "D4"
+		(property "Reference" "5V"
 			(at 0 -1.43 90)
 			(layer "F.SilkS")
@@
 		(descr "LED SMD 0603 (1608 Metric), square (rectangular) end terminal, IPC_7351 nominal, (Body size source: http://www.tortai-tech.com/upload/download/2011102023233369053.pdf), generated with kicad-footprint-generator")
 		(tags "LED")
-		(property "Reference" "D3"
+		(property "Reference" "12V"
 			(at 0 -1.43 90)
 			(layer "F.SilkS")
@@
 		(descr "LED SMD 0603 (1608 Metric), square (rectangular) end terminal, IPC_7351 nominal, (Body size source: http://www.tortai-tech.com/upload/download/2011102023233369053.pdf), generated with kicad-footprint-generator")
 		(tags "LED")
-		(property "Reference" "D5"
+		(property "Reference" "3.3V"
 			(at 0 -1.43 90)
 			(layer "F.SilkS")
