File: Ritsumori cup2026/Substrate/Motor driver board_1.0/Motor driver board_1.0.kicad_pcb (KiCad board)
At the start: 2 copper layers, 54.1 x 63.9 mm, 49 parts, among them J1 main, U1 DRV8412, U2 DRV8412

Commit message: Auto Backup: 2026/02/19 16:55:47.94
Parts:
- R3, R5: value 30k -> 1
Changed lines of the file:
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@@
 		(sheetname "/")
 		(sheetfile "Motor driver board_1.0.kicad_sch")
-		(attr through_hole)
+		(attr through_hole exclude_from_pos_files exclude_from_bom)
 		(fp_line
 			(start 1.49 1.04)
@@
 			)
 		)
-		(property "Value" "30k"
+		(property "Value" "1"
 			(at 0 1.43 0)
 			(layer "F.Fab")
@@
 			)
 		)
-		(property "Value" "30k"
+		(property "Value" "1"
 			(at 0 1.43 0)
 			(layer "F.Fab")
@@
 			)
 		)
+		(property "LCSC" "C22936"
+			(at 0 0 0)
+			(layer "F.SilkS")
+			(hide yes)
+			(effects
+				(font
+					(size 1.27 1.27)
+					(thickness 0.15)
+				)
+			)
+		)
 		(property ki_fp_filters "R_*")
 		(sheetname "/")
@@
 			(hide yes)
 			(effects
+				(font
+					(size 1.27 1.27)
+					(thickness 0.15)
+				)
+			)
+		)
+		(property "LCSC" ""
+			(at 0 0 0)
+			(layer "F.SilkS")
+			(hide yes)
+			(effects

Commit message: Auto Backup: 2026/03/24 15:00:23.58
Parts:
- removed U1, U2: DRV8412, Package_SO:HTSSOP-44-1EP_6.1x14mm_P0.635mm_EP5.2x14mm_Mask4.31x8.26mm_ThermalVias
- added 12V: Conn_01x01_Socket, TestPoint:TestPoint_Keystone_5000-5004_Miniature, F.Cu at (154.0, 90.0)
- added 3.3V: Conn_01x01_Socket, TestPoint:TestPoint_Keystone_5000-5004_Miniature, F.Cu at (154.0, 95.0)
- added FAULT1: Conn_01x01_Socket, TestPoint:TestPoint_Keystone_5000-5004_Miniature, F.Cu at (154.0, 100.0)
- added FAULT2: Conn_01x01_Socket, TestPoint:TestPoint_Keystone_5000-5004_Miniature, F.Cu at (154.0, 105.0)
- added GND: Conn_01x01_Socket, TestPoint:TestPoint_Keystone_5000-5004_Miniature, F.Cu at (154.0, 110.0)
- added IC1: DRV8412DDWR, Package_SO:HTSSOP-44-1EP_6.1x14mm_P0.635mm_EP5.2x14mm_Mask4.31x8.26mm, F.Cu at (170.0, 90.0)
- added IC2: DRV8412DDWR, Package_SO:HTSSOP-44-1EP_6.1x14mm_P0.635mm_EP5.2x14mm_Mask4.31x8.26mm, F.Cu at (170.0, 110.0)
- added R11: 30k, Resistor_SMD:R_0603_1608Metric, F.Cu at (177.0, 108.2)
- added R12: 3.3, Resistor_SMD:R_0603_1608Metric, F.Cu at (172.0, 124.0)
- C1: value 1 -> 330; footprint Capacitor_SMD:C_0603_1608Metric -> Capacitor_THT:CP_Radial_D10.0mm_P5.00mm
- C17: value 0.1u -> 10nF
- C18: value 0.1u -> 1000; footprint Capacitor_SMD:C_0603_1608Metric -> Capacitor_THT:CP_Radial_D10.0mm_P5.00mm
- C19: value 47 -> 330; footprint Capacitor_THT:CP_Radial_D6.3mm_P2.50mm -> Capacitor_THT:CP_Radial_D10.0mm_P5.00mm
- C20: value 1 -> 47; footprint Capacitor_SMD:C_0603_1608Metric -> Capacitor_THT:CP_Radial_D6.3mm_P2.50mm
- C21, C7: value 330 -> 0.1u; footprint Capacitor_THT:CP_Radial_D10.0mm_P5.00mm -> Capacitor_SMD:C_0603_1608Metric
- C22, C24, C25, C26, C3, C4, C5, C6: value 1 -> 0.1u
- C35: value 10n -> 10nF
- C8: value 1000 -> 0.1u; footprint Capacitor_THT:CP_Radial_D10.0mm_P5.00mm -> Capacitor_SMD:C_0603_1608Metric
- C9: value 10n -> 0.1u
- R1: value 3.3 -> 30k
- R10, R4: value 30k -> 1
- R3: value 1 -> 10k
- R5: value 1 -> 30k
- R9: value 30k -> 10k
- moved R6 54.5 mm to (172.0, 76.0)
- moved C7 35.0 mm to (162.0, 94.8)
- moved R7 32.4 mm to (177.0, 114.0), turned to 0 degrees
- moved C9 28.2 mm to (163.5, 97.5), turned to -90 degrees
- moved C21 27.1 mm to (177.0, 103.0), turned to 180 degrees
- moved R5 26.4 mm to (177.0, 88.5)
- moved R1 25.5 mm to (177.0, 94.0), turned to 0 degrees
- moved C14 25.3 mm to (158.5, 89.2), turned to -90 degrees
- moved R4 24.8 mm to (181.5, 88.5), turned to 0 degrees
- moved C4 21.0 mm to (180.0, 95.0), turned to -90 degrees
- moved C1 20.5 mm to (190.5, 74.0), turned to 0 degrees
- moved C34 19.7 mm to (163.5, 102.5), turned to -90 degrees
- moved C18 19.2 mm to (163.0, 74.0), turned to 180 degrees
- moved R8 19.0 mm to (177.0, 106.3), turned to 180 degrees
- moved C8 17.2 mm to (162.0, 91.0)
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- renumbered J1 to J6
Connections:
- C1 pad 1: GND -> VDD
- C1 pad 2: VDD -> GND
- C10 pad 1: GND -> +12V
- C10 pad 2: +12V -> GND
- C12 pad 1: +12V -> Motor2_B
- C12 pad 2: GND -> Net-(IC1-BST_D)
- C13 pad 1: GND -> Motor2_A
- C13 pad 2: +12V -> Net-(IC1-BST_C)
- C14 pad 1: Net-(U2-VREG) -> Motor1_B
- C14 pad 2: Net-(U2-AGND) -> Net-(IC1-BST_B)
- C16 pad 1: Motor1_B -> GND
- C16 pad 2: Net-(U2-BST_B) -> VDD
- C17 pad 1: Motor2_A -> GND
- C17 pad 2: Net-(U2-BST_C) -> Net-(C17-Pad2)
- C18 pad 1: Motor2_B -> +12V
- C18 pad 2: Net-(U2-BST_D) -> GND
- C20 pad 1: GND -> VDD
- C20 pad 2: VDD -> GND
- C21 pad 1: VDD -> GND
- C21 pad 2: GND -> VDD
- C23 pad 2: Net-(U1-AGND) -> Net-(IC2-AGND)
- C24 pad 1: GND -> VDD
- C24 pad 2: VDD -> GND
- C25 pad 2: VDD -> +12V
- C26 pad 1: GND -> +12V
- C26 pad 2: VDD -> GND
- C27 pad 1: +12V -> VDD
- C28 pad 1: GND -> +12V
- C28 pad 2: +12V -> GND
- C30 pad 1: GND -> Motor4_B
- C30 pad 2: +12V -> Net-(IC2-BST_D)
- C31 pad 1: Motor3_A -> Motor4_A
- C33 pad 1: Motor4_A -> Motor3_A
- C34 pad 1: Motor4_B -> GND
- C34 pad 2: Net-(U1-BST_D) -> VDD
- C35 pad 1: Net-(C35-Pad1) -> GND
- C35 pad 2: GND -> Net-(C35-Pad2)
- C5 pad 1: GND -> Net-(IC1-VREG)
- C5 pad 2: VDD -> Net-(IC1-AGND)
- C6 pad 1: GND -> VDD
- C6 pad 2: VDD -> GND
- C7 pad 1: VDD -> GND
- C7 pad 2: GND -> +12V
- C9 pad 1: Net-(C9-Pad1) -> VDD
- R1 pad 1: +12V -> Net-(IC1-~{RESET_CD})
- R1 pad 2: Net-(C9-Pad1) -> VDD
- R10 pad 1: VDD -> GND
- R10 pad 2: Net-(U1-~{RESET_AB}) -> Net-(IC2-AGND)
- R2 pad 1: Net-(U2-AGND) -> VDD
- R3 pad 1: GND -> FAULT1
- R3 pad 2: Net-(U2-AGND) -> VDD
- R4 pad 1: Net-(U1-AGND) -> GND
- R4 pad 2: Net-(U1-OC_ADJ) -> Net-(IC1-AGND)
- R5 pad 1: GND -> Net-(IC1-OC_ADJ)
- R5 pad 2: Net-(U1-AGND) -> Net-(IC1-AGND)
- R6 pad 2: Net-(C35-Pad1) -> Net-(C17-Pad2)
- R7 pad 1: VDD -> Net-(IC2-~{RESET_CD})
- R7 pad 2: Net-(U2-~{RESET_AB}) -> VDD
- R8 pad 1: Net-(U2-~{RESET_CD}) -> VDD
- R8 pad 2: VDD -> Net-(IC2-~{RESET_AB})
- R9 pad 1: Net-(U1-~{RESET_CD}) -> FAULT2
Routing:
- net VDD: track 242.8 -> 350.2 mm, vias 1 -> 2
- net FAULT1: track 0.00 -> 45.2 mm, vias 0 -> 3
- net FAULT2: track 0.00 -> 28.4 mm, vias 0 -> 1
- net Motor4_B: track 54.6 -> 79.0 mm, vias 3 -> 5
- net Net-(U1-AGND): track 21.1 -> 0.00 mm, vias 2 -> 0
- net Net-(IC2-AGND): track 0.00 -> 21.1 mm, vias 0 -> 2
- net Net-(U2-AGND): track 20.9 -> 0.00 mm, vias 2 -> 0
- net Net-(IC1-AGND): track 0.00 -> 20.6 mm, vias 0 -> 2
- net Motor2_B: track 88.6 -> 75.4 mm, vias 2 -> 5
- net +12V: track 197.0 -> 209.9 mm
- net Net-(U2-VREG): track 12.9 -> 0.00 mm, vias 2 -> 0
- net Motor3_B: track 82.9 -> 95.2 mm, vias 3 -> 5
- net Motor4_A: track 76.7 -> 86.3 mm, vias 3 -> 5
- net Net-(U2-BST_C): track 8.88 -> 0.00 mm, vias 2 -> 0
- net Motor1_A: track 49.6 -> 58.3 mm, vias 2 -> 3
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