File: Ritsumori cup2026/Substrate/Main board/Main board.kicad_pcb (KiCad board)
At the start: 2 copper layers, 67.4 x 39.2 mm, 17 parts, among them IC1 STM32F446RET6, J1 main_PC, J2 Conn_02x10_Odd_Even, J3 Conn_02x10_Odd_Even, J5 Conn_01x04_Pin, J6 Conn_01x04_Pin, SW1 SW_Push

Commit message: Auto Backup: 2026/02/19 18:25:14.96
Connections:
- J2 pad 17: +12V -> VDD
- J2 pad 18: VDD -> +12V
- J6 pad 2: unconnected-(J6-Pin_2-Pad2) -> GND
- J6 pad 3: GND -> unconnected-(J6-Pin_3-Pad3)
Routing:
- net VDD: track 181.9 -> 192.1 mm, vias 4 -> 5
- net +12V: track 26.6 -> 33.3 mm
- net SW: track 36.5 -> 37.6 mm

Commit message: Auto Backup: 2026/03/09 13:07:55.49
Parts:
- C6: value 22u -> 4.7u
Changed lines of the file:
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@@
 			)
 		)
-		(property "Value" "22u"
+		(property "Value" "4.7u"
 			(at 0 1.43 90)
 			(layer "F.Fab")

Commit message: Auto Backup: 2026/04/13 16:29:43.37
Connections:
- J2 pad 17: VDD -> +12V
Routing:
- net VDD: track 192.1 -> 179.3 mm, vias 5 -> 4
- net +12V: track 33.3 -> 35.8 mm
Changed lines of the file:
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@@
 			(layers "*.Cu" "*.Mask")
 			(remove_unused_layers no)
-			(net 2 "VDD")
+			(net 21 "+12V")
 			(pinfunction "Pin_17")
 			(pintype "passive")
@@
 	)
 	(segment
-		(start 84.825 63.175)
-		(end 84.825 62.315)
-		(width 0.3)
-		(layer "F.Cu")
-		(net 2)
-	)
-	(segment
 		(start 49.67 36.06)
 		(end 49.67 36.42)
@@
 	)
 	(segment
-		(start 84.825 62.315)
-		(end 81.4 58.89)
-		(width 0.3)
-		(layer "F.Cu")
-		(net 2)
-	)
-	(segment
 		(start 49.67 46.04)
 		(end 49.67 47)
@@
 	)
 	(via
-		(at 84.825 63.175)
-		(size 0.6)
-		(drill 0.3)
-		(layers "F.Cu" "B.Cu")
-		(net 2)
-	)
-	(via
 		(at 71.68 37)
 		(size 0.6)
@@
 	)
 	(segment
-		(start 90.965 65.565)
-		(end 87.215 65.565)
-		(width 0.3)
-		(layer "B.Cu")
-		(net 2)
-	)
-	(segment
 		(start 88.95 67.58)
 		(end 90.965 65.565)
@@
 		(start 75.67 65.62)
 		(end 77.63 67.58)
-		(width 0.3)
-		(layer "B.Cu")
-		(net 2)
-	)
-	(segment
-		(start 87.215 65.565)
-		(end 84.825 63.175)
 		(width 0.3)
 		(layer "B.Cu")
@@
 		(width 1)
 		(layer "F.Cu")
+		(net 21)
+	)
+	(segment
+		(start 78.86 58.89)
+		(end 81.4 58.89)
+		(width 1)
+		(layer "F.Cu")
