File: Ritsumori cup2026/Substrate/Main board/Main board.kicad_sch (KiCad schematic)
At the start: 17 parts, among them IC1 STM32F446RET6, J1 main_PC, J2 Conn_02x10_Odd_Even, J3 Conn_02x10_Odd_Even, J5 Conn_01x04_Pin, J6 Conn_01x04_Pin, SW1 SW_Push

Commit message: Auto Backup: 2026/02/19 18:25:14.96
Connections:
- net +12V: now also J2.18 (Pin_18); no longer J2.17 (Pin_17)
- net GND: now also J6.2 (Pin_2); no longer J6.3 (Pin_3)
- net VDD: now also J2.17 (Pin_17); no longer J2.18 (Pin_18)
Changed lines of the file:
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@@
 	)
 	(no_connect
-		(at 262.89 73.66)
+		(at 262.89 76.2)
 	)
 	(no_connect
@@
 	(symbol
 		(lib_id "power:GND")
-		(at 262.89 76.2 90)
+		(at 262.89 73.66 90)
 		(unit 1)
 		(exclude_from_sim no)
@@
 		(fields_autoplaced yes)
 		(property "Reference" "#PWR028"
-			(at 269.24 76.2 0)
+			(at 269.24 73.66 0)
 			(effects
 				(font
@@
 		)
 		(property "Value" "GND"
-			(at 266.7 76.1999 90)
+			(at 266.7 73.6599 90)
 			(effects
 				(font
@@
 		)
 		(property "Footprint" ""
-			(at 262.89 76.2 0)
+			(at 262.89 73.66 0)
 			(effects
 				(font
@@
 		)
 		(property "Datasheet" ""
-			(at 262.89 76.2 0)
+			(at 262.89 73.66 0)
 			(effects
 				(font
@@
 		)
 		(property "Description" "Power symbol creates a global label with name \"GND\" , ground"
-			(at 262.89 76.2 0)
+			(at 262.89 73.66 0)
 			(effects
 				(font
@@
 	(symbol
 		(lib_id "power:+12V")
-		(at 212.09 72.39 90)
-		(mirror x)
+		(at 224.79 72.39 270)
 		(unit 1)
 		(exclude_from_sim no)
@@
 		(fields_autoplaced yes)
 		(property "Reference" "#PWR019"
-			(at 215.9 72.39 0)
+			(at 220.98 72.39 0)
 			(effects
 				(font
@@
 		)
 		(property "Value" "+12V"
-			(at 208.28 72.3899 90)
+			(at 228.6 72.3899 90)
 			(effects
 				(font
@@
 		)
 		(property "Footprint" ""
-			(at 212.09 72.39 0)
+			(at 224.79 72.39 0)
 			(effects
 				(font
@@
 		)
 		(property "Datasheet" ""
-			(at 212.09 72.39 0)
+			(at 224.79 72.39 0)
 			(effects
 				(font
@@
 		)
 		(property "Description" "Power symbol creates a global label with name \"+12V\""
-			(at 212.09 72.39 0)
+			(at 224.79 72.39 0)
 			(effects
 				(font
@@
 	(symbol
 		(lib_id "power:VDD")
-		(at 224.79 72.39 270)
-		(mirror x)
+		(at 212.09 72.39 90)
 		(unit 1)
 		(exclude_from_sim no)
@@
 		(fields_autoplaced yes)
 		(property "Reference" "#PWR017"
-			(at 220.98 72.39 0)
+			(at 215.9 72.39 0)
 			(effects
 				(font
@@
 		)
 		(property "Value" "VDD"
-			(at 228.6 72.3899 90)
+			(at 208.28 72.3899 90)
 			(effects
 				(font
@@
 		)
 		(property "Footprint" ""
-			(at 224.79 72.39 0)
+			(at 212.09 72.39 0)
 			(effects
 				(font
@@
 		)
 		(property "Datasheet" ""
-			(at 224.79 72.39 0)
+			(at 212.09 72.39 0)
 			(effects
 				(font
@@
 		)
 		(property "Description" "Power symbol creates a global label with name \"VDD\""
-			(at 224.79 72.39 0)
+			(at 212.09 72.39 0)
 			(effects
 				(font

Commit message: Auto Backup: 2026/03/09 13:07:55.49
Parts:
- C6: value 22u -> 4.7u
Changed lines of the file:
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@@
 			)
 		)
-		(property "Value" "22u"
+		(property "Value" "4.7u"
 			(at 117.094 161.29 0)
 			(effects

Commit message: Auto Backup: 2026/04/13 16:29:43.37
Connections:
- net +12V: now also J2.17 (Pin_17)
- net VDD: no longer J2.17 (Pin_17)
Changed lines of the file:
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@@
-	)
-	(symbol
-		(lib_id "power:VDD")
-		(at 212.09 72.39 90)
-		(unit 1)
-		(exclude_from_sim no)
-		(in_bom yes)
-		(on_board yes)
-		(dnp no)
-		(fields_autoplaced yes)
-		(property "Reference" "#PWR017"
-			(at 215.9 72.39 0)
-			(effects
-				(font
-					(size 1.27 1.27)
-				)
-				(hide yes)
-			)
-		)
-		(property "Value" "VDD"
-			(at 208.28 72.3899 90)
-			(effects
-				(font
-					(size 1.27 1.27)
-				)
-				(justify left)
-			)
-		)
-		(property "Footprint" ""
-			(at 212.09 72.39 0)
-			(effects
-				(font
-					(size 1.27 1.27)
-				)
-				(hide yes)
-			)
-		)
-		(property "Datasheet" ""
-			(at 212.09 72.39 0)
-			(effects
-				(font
-					(size 1.27 1.27)
-				)
-				(hide yes)
-			)
-		)
-		(property "Description" "Power symbol creates a global label with name \"VDD\""
-			(at 212.09 72.39 0)
-			(effects
-				(font
-					(size 1.27 1.27)
-				)
-				(hide yes)
-			)
-		)
-		(pin "1"
-		)
-		(instances
-			(project ""
-				(path "/69cb4efb-39ce-4105-ae0c-29d9feedd3fe"
-					(reference "#PWR017")
-					(unit 1)
-				)
-			)
-		)
 	)
 	(symbol
@@
 					(unit 1)
 				)
+			)
+		)
+	)
+	(symbol
+		(lib_id "power:+12V")
+		(at 212.09 72.39 90)
+		(unit 1)
+		(exclude_from_sim no)
+		(in_bom yes)
+		(on_board yes)
+		(dnp no)
+		(fields_autoplaced yes)
+		(property "Reference" "#PWR012"
+			(at 215.9 72.39 0)
+			(effects
+				(font
+					(size 1.27 1.27)
+				)
+				(hide yes)
+			)
+		)
+		(property "Value" "+12V"
+			(at 208.28 72.3899 90)
+			(effects
+				(font
+					(size 1.27 1.27)
+				)
+				(justify left)
+			)
+		)
+		(property "Footprint" ""
+			(at 212.09 72.39 0)
+			(effects
+				(font
+					(size 1.27 1.27)
+				)
+				(hide yes)
+			)
+		)
+		(property "Datasheet" ""
+			(at 212.09 72.39 0)
+			(effects
+				(font
+					(size 1.27 1.27)
+				)
+				(hide yes)
+			)
+		)
+		(property "Description" "Power symbol creates a global label with name \"+12V\""
+			(at 212.09 72.39 0)
+			(effects
+				(font
+					(size 1.27 1.27)
+				)
+				(hide yes)
+			)
+		)
+		(pin "1"
+		)
+		(instances
+			(project "Main board"
+				(path "/69cb4efb-39ce-4105-ae0c-29d9feedd3fe"
+					(reference "#PWR012")
+					(unit 1)
+				)
