File: NEST2026/Substrate/Motor driver board_1.0/Motor driver board_1.0.kicad_pcb (KiCad board)
At the start: 2 copper layers, 50 x 64 mm, 54 parts, among them IC1 DRV8412DDWR, IC2 DRV8412DDWR, J1 Conn_01x02_Socket, J2 Conn_01x02_Socket, J3 Conn_01x02_Socket, J4 Conn_01x02_Socket, J5 Conn_01x02_Socket, J6 Conn_01x08_Socket

Commit message: Auto Backup: 2026/04/29 17:42:26.28
Routing:
- net GND: vias 50 -> 81
